File: PCB/numpad - plate.kicad_pcb (KiCad board)
At the start: 2 copper layers, 105.6 x 115.1 mm, 0 parts

Commit message: Exported gerbers
Other:
- outline, holes or cut-outs redrawn
Changed lines of the file:
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@@
       (drillshape 0)
       (scaleselection 1)
-      (outputdirectory "Gerber/"))
+      (outputdirectory "Gerber/Plate/"))
   )
   (net 0 "")
@@
     (uvia_drill 0.1)
   )
-  (gr_line (start 155.96205 131.35735) (end 155.96205 100.0062) (layer Edge.Cuts) (width 0.05))
-  (gr_line (start 139.6912 60.3212) (end 157.54945 60.3212) (layer Edge.Cuts) (width 0.05))
-  (gr_arc (start 157.54945 63.496) (end 160.72425 63.496) (angle -90) (layer Edge.Cuts) (width 0.05))
-  (gr_line (start 160.72425 98.4188) (end 160.72425 63.496) (layer Edge.Cuts) (width 0.05))
-  (gr_arc (start 159.93055 98.4188) (end 159.93055 99.2125) (angle -90) (layer Edge.Cuts) (width 0.05))
-  (gr_line (start 156.75575 99.2125) (end 159.93055 99.2125) (layer Edge.Cuts) (width 0.05))
-  (gr_arc (start 156.75575 100.0062) (end 156.75575 99.2125) (angle -90) (layer Edge.Cuts) (width 0.05))
+  (gr_line (start 139.6912 60.3212) (end 158.74 60.3212) (layer Edge.Cuts) (width 0.05))
+  (gr_line (start 156.3589 103.181) (end 161.1211 103.181) (layer Edge.Cuts) (width 0.05))
+  (gr_line (start 161.9148 63.496) (end 161.9148 102.3873) (layer Edge.Cuts) (width 0.05))
+  (gr_line (start 155.5652 131.35735) (end 155.5652 103.9747) (layer Edge.Cuts) (width 0.05))
+  (gr_line (start 156.3589 132.15105) (end 183.3447 132.15105) (layer Edge.Cuts) (width 0.05))
+  (gr_arc (start 158.74 63.496) (end 161.9148 63.496) (angle -90) (layer Edge.Cuts) (width 0.05))
+  (gr_arc (start 161.1211 102.3873) (end 161.1211 103.181) (angle -90) (layer Edge.Cuts) (width 0.05))
+  (gr_arc (start 156.3589 103.9747) (end 156.3589 103.181) (angle -90) (layer Edge.Cuts) (width 0.05))
   (gr_line (start 184.1384 132.94475) (end 184.1384 172.2329) (layer Edge.Cuts) (width 0.05))
   (gr_arc (start 183.3447 132.94475) (end 184.1384 132.94475) (angle -90) (layer Edge.Cuts) (width 0.05))
-  (gr_line (start 156.75575 132.15105) (end 183.3447 132.15105) (layer Edge.Cuts) (width 0.05))
-  (gr_arc (start 156.75575 131.35735) (end 155.96205 131.35735) (angle -90) (layer Edge.Cuts) (width 0.05))
+  (gr_arc (start 156.3589 131.35735) (end 155.5652 131.35735) (angle -90) (layer Edge.Cuts) (width 0.05))
   (gr_poly (pts (xy 138.50065 81.35425) (xy 138.1038 82.14795) (xy 138.1038 95.64085) (xy 138.50065 96.43455) (xy 139.29435 96.8314) (xy 152.78725 96.8314) (xy 153.58095 96.43455) (xy 153.9778 95.64085) (xy 153.9778 82.14795) (xy 153.58095 81.35425) (xy 152.78725 80.9574) (xy 139.29435 80.9574)) (layer B.Mask) (width 0.1))
   (gr_poly (pts (xy 119.45185 138.50065) (xy 119.055 139.29435) (xy 119.055 152.78725) (xy 119.45185 153.58095) (xy 120.24555 153.9778) (xy 133.73845 153.9778) (xy 134.53215 153.58095) (xy 134.929 152.78725) (xy 134.929 139.29435) (xy 134.53215 138.50065) (xy 133.73845 138.1038) (xy 120.24555 138.1038)) (layer B.Mask) (width 0.1))
