File: PCB/numpad.kicad_sch (KiCad schematic)
At the start: 53 parts, among them J1 AVR-ISP-6, J2 Conn_01x04_Female, SW1 SW_Push, U1 ProMicro

Commit message: Curved more traces
Parts:
- removed R2: 10k, Resistor_SMD:R_0603_1608Metric, symbol Device:R_Small
Changed lines of the file:
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@@
   (junction (at 209.55 86.36) (diameter 0) (color 0 0 0 0)
-  )
-  (junction (at 111.76 99.06) (diameter 0) (color 0 0 0 0)
   )
   (junction (at 176.53 86.36) (diameter 0) (color 0 0 0 0)
@@
     (stroke (width 0) (type default) (color 0 0 0 0))
   )
-  (wire (pts (xy 111.76 99.06) (xy 111.76 96.52))
-    (stroke (width 0) (type default) (color 0 0 0 0))
-  )
   (wire (pts (xy 181.61 96.52) (xy 179.07 96.52))
     (stroke (width 0) (type default) (color 0 0 0 0))
@@
     (stroke (width 0) (type default) (color 0 0 0 0))
   )
-  (wire (pts (xy 106.68 99.06) (xy 111.76 99.06))
+  (wire (pts (xy 106.68 99.06) (xy 118.11 99.06))
     (stroke (width 0) (type default) (color 0 0 0 0))
   )
@@
   )
   (wire (pts (xy 165.1 77.47) (xy 162.56 77.47))
-    (stroke (width 0) (type default) (color 0 0 0 0))
-  )
-  (wire (pts (xy 118.11 99.06) (xy 111.76 99.06))
     (stroke (width 0) (type default) (color 0 0 0 0))
   )
@@
     )
     (property "Datasheet" "" (id 3) (at 129.54 101.6 0)
-      (effects (font (size 1.27 1.27)) hide)
-    )
-    (pin "1")
-  )
-  (symbol (lib_id "Device:R_Small") (at 111.76 93.98 0) (unit 1)
-    (in_bom yes) (on_board yes)
-    (property "Reference" "R2" (id 0) (at 113.2586 92.8116 0)
-      (effects (font (size 1.27 1.27)) (justify left))
-    )
-    (property "Value" "10k" (id 1) (at 113.2586 95.123 0)
-      (effects (font (size 1.27 1.27)) (justify left))
-    )
-    (property "Footprint" "Resistor_SMD:R_0603_1608Metric" (id 2) (at 111.76 93.98 0)
-      (effects (font (size 1.27 1.27)) hide)
-    )
-    (property "Datasheet" "~" (id 3) (at 111.76 93.98 0)
-      (effects (font (size 1.27 1.27)) hide)
-    )
-    (property "LCSC Part" "C25804" (id 4) (at 111.76 93.98 0)
-      (effects (font (size 1.27 1.27)) hide)
-    )
-    (pin "1")
-    (pin "2")
-  )
-  (symbol (lib_id "power:+5V") (at 111.76 91.44 0) (unit 1)
-    (in_bom yes) (on_board yes)
-    (property "Reference" "#PWR037" (id 0) (at 111.76 95.25 0)
-      (effects (font (size 1.27 1.27)) hide)
-    )
-    (property "Value" "+5V" (id 1) (at 112.141 87.0458 0))
-    (property "Footprint" "" (id 2) (at 111.76 91.44 0)
-      (effects (font (size 1.27 1.27)) hide)
-    )
-    (property "Datasheet" "" (id 3) (at 111.76 91.44 0)
       (effects (font (size 1.27 1.27)) hide)
     )
@@
       (reference "#PWR020") (unit 1) (value "GND") (footprint "")
     )
-    (path "/00000000-0000-0000-0000-000061993cbf"
-      (reference "#PWR037") (unit 1) (value "+5V") (footprint "")
-    )
     (path "/00000000-0000-0000-0000-00006198e7fb"
       (reference "#PWR041") (unit 1) (value "GND") (footprint "")
@@
       (reference "R1") (unit 1) (value "470") (footprint "Resistor_SMD:R_0603_1608Metric")
     )
-    (path "/00000000-0000-0000-0000-00006198ff4a"
-      (reference "R2") (unit 1) (value "10k") (footprint "Resistor_SMD:R_0603_1608Metric")
-    )
     (path "/6eedbfde-f698-4972-8341-01f795b14464/5eb001bc-ce47-477b-94e7-61cbfe22ed73"

Commit message: Updated numpad switch labels
Parts:
- MX1: value CherryMX -> Num
- MX10: value CherryMX -> 6
- MX11: value CherryMX -> +
- MX12: value CherryMX -> 1
- MX13: value CherryMX -> 2
- MX14: value CherryMX -> 3
- MX15: value CherryMX -> 0
- MX16: value CherryMX -> .
- MX17: value CherryMX -> Enter
- MX18: value CherryMX -> ALT
- MX2: value CherryMX -> /
- MX3: value CherryMX -> *
- MX4: value CherryMX -> 7
- MX5: value CherryMX -> 8
- MX6: value CherryMX -> 9
- MX7: value CherryMX -> -
- MX8: value CherryMX -> 4
- MX9: value CherryMX -> 5
